File: grbl-board.brd (EAGLE design)
At the start: 100 x 60 mm, 51 parts, among them IC1 MEGA328-P, IC2 FT232RL, IC3 ADuM1201AR, IC4 LM2596S, Q1 16 MHz, X1 PN61729-S

Commit message: ver.1.0
Parts:
- removed SV4: ISP, con-ml:ML6
- added C5, C6: (no value), adafruit:C0805K
- added COOLANT_EN: 22-23-2031, con-molex:22-23-2031
- added OK8: PC817, optocoupler:DIL04
- added R11: 1K, resistor:M0805
- SPINDLE: value 22-23-2041 -> 22-23-2031; device con-molex:22-23-2041 -> con-molex:22-23-2031
- moved R10 5.08 mm to (30.5, 44.1)
- moved OK7 5.08 mm to (27.3, 39.4)
- moved PROBE 5.08 mm to (27.3, 54.6)
- moved SV8 5.08 mm to (27.3, 48.3)
- moved R4 4.94 mm to (39.7, 20.3), turned to 0 degrees
- moved OK4 3.18 mm to (60.3, 39.4)
- moved R9 3.18 mm to (47.0, 44.1)
- moved RESET/ABORT 3.18 mm to (60.3, 54.6)
- moved SV5 3.18 mm to (60.3, 48.3)
- moved FEED_HOLD 3.17 mm to (52.1, 54.6)
- moved OK5 3.17 mm to (52.1, 39.4)
- moved OK6 3.17 mm to (43.8, 39.4)
- moved R7 3.17 mm to (63.5, 44.1)
- moved R8 3.17 mm to (55.2, 44.1)
- moved START/RESUME 3.17 mm to (43.8, 54.6)
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Connections:
- new net N$32: OK8.4, R11.1
- new net N$33: COOLANT_EN.1, R11.2
- net +24V: now also COOLANT_EN.3
- net COOLANT_EN: now also OK8.1; no longer SPINDLE.1
- net DGND: now also COOLANT_EN.2, OK8.3
- net GND: now also C5.1, C6.1, OK8.2, SPINDLE.3; no longer SPINDLE.4, SV4.6
- net N$6: now also C5.2
- net N$7: now also C6.2
- net RESET: no longer SV4.5
- net SPINDLE-DIR: now also SPINDLE.1; no longer SPINDLE.2, SV4.3
- net SPINDLE-PWM: now also SPINDLE.2; no longer SPINDLE.3, SV4.4
- net Z-LIMIT*: no longer SV4.1
Routing:
- net Z-LIMIT*: track 32.9 -> 7.83 mm
- net DGND: track 138.6 -> 160.1 mm
- net SPINDLE-PWM: track 50.5 -> 29.7 mm
- net +24V: track 158.0 -> 176.1 mm
- net COOLANT_EN: track 0.00 -> 17.1 mm
- net SPINDLE-DIR: track 49.4 -> 32.9 mm
- net GND: track 262.8 -> 273.0 mm
- net +5V: track 112.2 -> 122.3 mm
- net N$32: track 0.00 -> 8.26 mm
- net CYCLE_START/RESUME*: track 14.3 -> 9.67 mm
- net N$33: track 0.00 -> 3.83 mm
- net PROBE*: track 14.2 -> 17.5 mm
- net RESET/ABORT*: track 8.16 -> 9.66 mm
- net FEED_HOLD*: track 8.78 -> 7.62 mm
- net N$7: track 5.77 -> 6.68 mm
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Other:
- board text added: "GRBL board v.1.0"
